File: hardware/kicad/power.kicad_sch (KiCad schematic)
At the start: 0 parts

Commit message: kicad: add J1 power input terminal (24V+/GND/PE) to power sheet
Adds the 3-pin pluggable input terminal J1 (Phoenix MSTBA
2,5/3-G-5,08 footprint family). Pins 1/2/3 are wired to
+24V / GND / Earth_Protective power flags, each backed by
a PWR_FLAG sentinel so ERC sees the rails as externally
driven. Embeds the five required lib_symbols
(Screw_Terminal_01x03, +24V, GND, Earth_Protective,
PWR_FLAG) directly in power.kicad_sch as per KiCad 10
convention.

Footprint assignment is deferred to a later PCB-layout
chunk; the value field carries the intended part number
(Phoenix MSTBA 2,5/3-G-5,08, 5.08 mm pitch).

ERC passes 0/0 across all five sheets. Generation is
deterministic (bit-identical on consecutive runs).
Parts:
- added J1: Phoenix_MSTBA_2,5/3-G-5,08, symbol Connector:Screw_Terminal_01x03
Connections:
- new net +24V: J1.1 (Pin_1)
- new net Earth_Protective: J1.3 (Pin_3)
- new net GND: J1.2 (Pin_2)
