File: hardware/kicad/power.kicad_sch (KiCad schematic)
At the start: 26 parts, among them J1 Phoenix_MSTBA_2,5/3-G-5,08, Q1 PMV65XP, U1 LM2596S-5.0, U2 TPS62933

Commit message: kicad+docs: v0.17 - J1 24V terminal block placed at central cable-hole zone
Relocate J1 (Phoenix MSTBA 2,5/3-G-5,08) from the chord-edge connector
strip into the central PCB area, directly north of the Ø12 mm cable
pass-through hole. Removes one LED (D20) + its decoupling cap (C29)
from the AQI ring to open a corridor for the 24 V supply cable.

Geometry:
  - J1 PCB anchor (-5.08, -22.4), rotation 0.
  - Pin row at PCB Y=-22.4, pin 1=+24V at X=-5.08, pin 2=GND at X=0,
    pin 3=PE at X=+5.08. Body extends south to PCB Y=-12.29.
  - Cable enters connector mouth from south face; ~6.3-6.6 mm of
    horizontal travel for the cable bend from the hole exit.
  - ESP32 anchor_y shifted -24.70 -> -26.20 (1.5 mm north) to make
    room for J1's 13 mm courtyard depth between the LED ring's north
    corners and the ESP32 daughterboard's south edge.

LED ring v0.17 changes:
  - LED_RING_SKIP_INDICES = (9,) skips D20 in both PCB and schematic.
  - Daisy chain: D19.DOUT -> D21.DIN (5-segment route through the now-
    empty D20 row position in the schematic column).
  - Final ring has 11 LEDs (was 12 in v0.16).

PCB silkscreen:
  - "J1 (24V)" board-level F.SilkS label 6 mm west of the J1 body.
  - "24V"/"GND"/"PE" per-pin labels on F.Fab (silk-overlap-exempt).
  - In-footprint Reference/Value hidden to avoid silk_overlap with
    the ESP32 daughterboard south edge.

Schematic:
  - J1's Footprint property populated (was empty in v0.2). Datasheet
    and Description also filled in.
  - D20 + C29 schematic symbols and per-LED wires dropped.

DRC=0, ERC=0.

Co-Authored-By: Claude Opus 4.7 (1M context) <noreply@anthropic.com>
Parts:
- J1: footprint (none) -> Connector_Phoenix_MSTB:PhoenixContact_MSTBA_2,5_3-G-5,08_1x03_P5.08mm_Horizontal
Changed lines of the file:
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@@
 		)
 	)
-	(property "Footprint" ""
+	(property "Footprint" "Connector_Phoenix_MSTB:PhoenixContact_MSTBA_2,5_3-G-5,08_1x03_P5.08mm_Horizontal"
 		(at 57.15 86.36 0)
 		(effects
@@
 		)
 	)
-	(property "Datasheet" ""
+	(property "Datasheet" "https://www.phoenixcontact.com/online/portal/us?uri=pxc-oc-itemdetail:pid=1757255"
 		(at 57.15 86.36 0)
 		(effects
@@
 		)
 	)
-	(property "Description" ""
+	(property "Description" "Phoenix Contact MSTBA 2,5/3-G-5,08 — 3-pin 5.08 mm pitch pluggable terminal block base. 24 V supply input: pin 1 = +24V_unprotected, pin 2 = GND, pin 3 = PE. Mates with a Phoenix COMBICON 5.08 mm 3-pin plug. Order code 1757255 (12 A) or 1923872 (16 A HC)."
 		(at 57.15 86.36 0)
 		(effects

Commit message: kicad: v0.20 - C3 renumber HF-bypass caps C3b/C4b/C5b/C6b/C9b -> C13..C17
Pre-routing review v0.19 finding C3 (Critical): KiCad's BOM annotator
treats trailing-letter references like 'C3b' as un-annotated 'C3' + suffix
letter, emitting them as 'C3b?' on BOM export and breaking JLCPCB / Mouser
upload. Renamed in lockstep across schematic / wire labels / Python local
identifiers (no electrical change):

  C3b -> C13   (input HF bypass at U1.VIN)
  C4b -> C14   (output HF bypass at +5V)
  C5b -> C15   (input HF bypass at U2.VIN)
  C6b -> C16   (output HF bypass at +3V3)
  C9b -> C17   (HF decoupling at ESP32 +3V3)

ERC=0, DRC=0. BOM export verified: all five caps now appear as plain
"C13".."C17" with no '?' suffix.

Co-Authored-By: Claude Opus 4.7 (1M context) <noreply@anthropic.com>
Parts:
- removed C3b, C4b, C5b, C6b: 100nF, symbol Device:C
- added C13, C14, C15, C16: 100nF, symbol Device:C
Connections:
- net +24V: now also C13.1
- net +3V3: now also C16.1
- net +5V: now also C14.1, C15.1
- net GND: now also C13.2, C14.2, C15.2, C16.2
Changed lines of the file:
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@@
 	(dnp no)
 	(fields_autoplaced yes)
-	(property "Reference" "C3b"
+	(property "Reference" "C13"
 		(at 147.32 64.77 0)
 		(effects
@@
 		(project "oas"
 			(path "/515343fe-5590-5fd9-97ec-5bed0f979de2/1557665b-a568-58fc-b40f-759ed4998499"
-				(reference "C3b")
+				(reference "C13")
 				(unit 1)
 			)
@@
 	(dnp no)
 	(fields_autoplaced yes)
-	(property "Reference" "C4b"
+	(property "Reference" "C14"
 		(at 226.06 59.69 0)
 		(effects
@@
 		(project "oas"
 			(path "/515343fe-5590-5fd9-97ec-5bed0f979de2/1557665b-a568-58fc-b40f-759ed4998499"
-				(reference "C4b")
+				(reference "C14")
 				(unit 1)
 			)
@@
 	(dnp no)
 	(fields_autoplaced yes)
-	(property "Reference" "C5b"
+	(property "Reference" "C15"
 		(at 157.48 129.54 0)
 		(effects
@@
 		(project "oas"
 			(path "/515343fe-5590-5fd9-97ec-5bed0f979de2/1557665b-a568-58fc-b40f-759ed4998499"
-				(reference "C5b")
+				(reference "C15")
 				(unit 1)
 			)
@@
 	(dnp no)
 	(fields_autoplaced yes)
-	(property "Reference" "C6b"
+	(property "Reference" "C16"
 		(at 243.84 129.54 0)
 		(effects
@@
 		(project "oas"
 			(path "/515343fe-5590-5fd9-97ec-5bed0f979de2/1557665b-a568-58fc-b40f-759ed4998499"
-				(reference "C6b")
-				(unit 1)
-			)
+				(reference "C16")
+				(unit 1)
+			)

Commit message: kicad+docs: v0.24 - fix v0.23 regressions (lib-qualify footprints + ERC strict)
Closes review iteration 2 findings (`_review-iteration-2-v0.23.md`):

1. Mn3 V3 regression — lib-qualify footprint back-fill.
   `_build_pcb_ref_to_footprint()` now lib-qualifies bare PCB-side
   Footprint property values via a new `BARE_FOOTPRINT_TO_LIB` table
   (12 entries) and asserts every returned value contains `:`. In
   parallel, the inline `gen_*_pcb_footprint` generators that emitted
   bare names now write fully-qualified `Lib:Name` strings directly
   (`Capacitor_SMD:C_0402_1005Metric`, `Package_TO_SOT_SMD:SOT-23`,
   `Inductor_SMD:L_APV_ANR5040`, `Fuse:Fuse_2920_7451Metric`,
   `Capacitor_THT:CP_Radial_D8.0mm_P3.50mm`, etc.). 15 ERC
   `footprint_link_issues` warnings → 0.

2. Mj2 — `regenerate.py` ERC strict mode. `kicad-cli sch erc` now
   invoked with `--severity-error --severity-warning
   --exit-code-violations`, mirroring DRC strictness. Verified by
   corrupting a schematic Footprint property and confirming abort.
   CLAUDE.md "PCB design workflow" §3 ("aborts on any error or
   warning") is now actually enforced for ERC, not just DRC.

3. C1 V4 — derived `.kicad_pcb` / `.kicad_sch` resynced with
   `generate.py`. The v0.23 commit shipped `generate.py` updates
   without regenerating the derived files; this commit brings them
   into sync via `python regenerate.py`.

4. Mj1 — CLAUDE.md v0.23 changelog entry added retroactively
   (had been missing). v0.24 entry added documenting this fix
   series + the ERC-strictness lesson.

5. `hardware/components/_review-iteration-2-v0.23.md` committed
   (previously untracked).

DRC = 0 violations / 0 warnings.
ERC = 0 violations / 0 warnings (now strict).
Determinism self-check passes (17 files bit-identical across two
consecutive `regenerate.py` runs).

Co-Authored-By: Claude Opus 4.7 (1M context) <noreply@anthropic.com>
Parts:
- C1, C3: footprint (none) -> Capacitor_THT:CP_Radial_D8.0mm_P3.50mm
- C4: footprint (none) -> Capacitor_THT:CP_Radial_D6.3mm_P2.50mm
- Q1: footprint (none) -> Package_TO_SOT_SMD:SOT-23
Changed lines of the file:
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@@
 		)
 	)
-	(property "Footprint" ""
+	(property "Footprint" "Package_TO_SOT_SMD:SOT-23"
 		(at 82.55 78.74 0)
 		(effects
@@
 		)
 	)
-	(property "Footprint" ""
+	(property "Footprint" "Capacitor_THT:CP_Radial_D8.0mm_P3.50mm"
 		(at 111.76 66.04 0)
 		(effects
@@
 		)
 	)
-	(property "Footprint" ""
+	(property "Footprint" "Capacitor_THT:CP_Radial_D8.0mm_P3.50mm"
 		(at 129.54 66.04 0)
 		(effects
@@
 		)
 	)
-	(property "Footprint" ""
+	(property "Footprint" "Capacitor_THT:CP_Radial_D6.3mm_P2.50mm"
 		(at 208.28 60.96 0)
 		(effects

Commit message: kicad: v0.25 - widen Mn3 back-fill regex to capture indented footprint blocks
Closes review-iteration-3 (Mn3-residual + Nt-doc-comment) at v0.24:

- _build_pcb_ref_to_footprint() regex (?m)^\(footprint "..." widened to
  (?m)^\s*\(footprint "..." . KiCad pretty-prints some (footprint ...) blocks
  in oas.kicad_pcb with leading tab/space indentation; the column-0 anchor
  silently skipped 31 of 76 placed footprints in v0.24, leaving 27 schematic
  real-component symbols with empty Footprint properties (ERC-silent but
  cosmetically wrong). Match count: 45 -> 76 (exactly equal to kiutils
  enumeration). Verified no nested (footprint "..." references exist.
- Inner re.match relaxed to re.search since sliced blocks can begin with
  whitespace.
- Docstring updated to disclose the regex behavior honestly (closes
  Nt-doc-comment from review iter-3).
- All 65 real-component schematic instances now carry a fully-qualified
  Lib:Name Footprint property. Empty-Footprint count: 0 (was 27 at v0.24,
  51 at v0.22). Previously-missed refs now lib-qualified: C2 + C5-C17, D1-D3,
  F1, L1-L2, R1-R7, plus ZT1-ZT4.
- DRC = 0/0, ERC = 0/0, determinism self-check passes (17 files bit-identical
  across two consecutive runs). PCB geometry unchanged - schematic-side
  .kicad_sch diffs only.
- Adds the iteration-3 review file (hardware/components/_review-iteration-3-v0.24.md).

Co-Authored-By: Claude Opus 4.7 (1M context) <noreply@anthropic.com>
Parts:
- C13, C14, C15, C16, C7, C8: footprint (none) -> Capacitor_SMD:C_0603_1608Metric
- C2, C5, C6: footprint (none) -> Capacitor_SMD:C_0805_2012Metric
- D1: footprint (none) -> Diode_SMD:D_SMB
- D2: footprint (none) -> Diode_SMD:D_SMA
- D3: footprint (none) -> Diode_SMD:D_SOD-323
- F1: footprint (none) -> Fuse:Fuse_2920_7451Metric
- L1, L2: footprint (none) -> Inductor_SMD:L_APV_ANR5040
- R1, R2, R3, R4: footprint (none) -> Resistor_SMD:R_0603_1608Metric
Changed lines of the file:
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@@
 		)
 	)
-	(property "Footprint" ""
+	(property "Footprint" "Diode_SMD:D_SMB"
 		(at 66.04 87.63 0)
 		(effects
@@
 		)
 	)
-	(property "Footprint" ""
+	(property "Footprint" "Diode_SMD:D_SOD-323"
 		(at 72.39 88.9 0)
 		(effects
@@
 		)
 	)
-	(property "Footprint" ""
+	(property "Footprint" "Fuse:Fuse_2920_7451Metric"
 		(at 85.09 66.04 0)
 		(effects
@@
 		)
 	)
-	(property "Footprint" ""
+	(property "Footprint" "Resistor_SMD:R_0603_1608Metric"
 		(at 77.47 99.06 90)
 		(effects
@@
 		)
 	)
-	(property "Footprint" ""
+	(property "Footprint" "Resistor_SMD:R_0603_1608Metric"
 		(at 77.47 88.9 90)
 		(effects
@@
 		)
 	)
-	(property "Footprint" ""
+	(property "Footprint" "Capacitor_SMD:C_0805_2012Metric"
 		(at 30.48 109.22 0)
 		(effects
@@
 		)
 	)
-	(property "Footprint" ""
+	(property "Footprint" "Inductor_SMD:L_APV_ANR5040"
 		(at 193.04 60.96 0)
 		(effects
@@
 		)
 	)
-	(property "Footprint" ""
+	(property "Footprint" "Diode_SMD:D_SMA"
 		(at 187.96 71.12 0)
 		(effects
@@
 		)
 	)
-	(property "Footprint" ""
+	(property "Footprint" "Capacitor_SMD:C_0603_1608Metric"
 		(at 144.78 66.04 0)
 		(effects
@@
 		)
 	)
-	(property "Footprint" ""
+	(property "Footprint" "Capacitor_SMD:C_0603_1608Metric"
 		(at 223.52 60.96 0)
 		(effects
@@
 		)
 	)
-	(property "Footprint" ""
+	(property "Footprint" "Inductor_SMD:L_APV_ANR5040"
 		(at 195.58 130.81 0)
 		(effects
@@
 		)
 	)
-	(property "Footprint" ""
+	(property "Footprint" "Capacitor_SMD:C_0805_2012Metric"
 		(at 139.7 130.81 0)
 		(effects
@@
 		)
 	)
-	(property "Footprint" ""
+	(property "Footprint" "Capacitor_SMD:C_0603_1608Metric"
 		(at 154.94 130.81 0)
 		(effects
@@
 		)
 	)
-	(property "Footprint" ""
+	(property "Footprint" "Capacitor_SMD:C_0805_2012Metric"
 		(at 226.06 130.81 0)
 		(effects
@@
 		)
 	)
-	(property "Footprint" ""
+	(property "Footprint" "Capacitor_SMD:C_0603_1608Metric"
 		(at 241.3 130.81 0)
 		(effects
@@
 		)
 	)
-	(property "Footprint" ""
+	(property "Footprint" "Capacitor_SMD:C_0603_1608Metric"
 		(at 182.88 130.81 0)
 		(effects
@@
 		)
 	)
-	(property "Footprint" ""
+	(property "Footprint" "Capacitor_SMD:C_0603_1608Metric"
 		(at 161.29 140.97 0)
 		(effects
@@
 		)
 	)
-	(property "Footprint" ""
+	(property "Footprint" "Resistor_SMD:R_0603_1608Metric"
 		(at 209.55 138.43 90)
 		(effects
@@
 		)
 	)
-	(property "Footprint" ""
+	(property "Footprint" "Resistor_SMD:R_0603_1608Metric"
 		(at 209.55 146.05 90)
 		(effects
