File: hardware/kicad/power.kicad_sch (KiCad schematic)
At the start: 26 parts, among them J1 Phoenix_MSTBA_2,5/3-G-5,08, Q1 AO3401A, U1 LM2596S-5.0, U2 TPS62933

Commit message: fix(boardgen): LED ring emission outward, F1 1812 downsize, J1 no-go zone
LED ring (SK6812-SIDE D11..D18):
- Flip rotation formula (270-theta) -> (90-theta) so emission face points
  radially OUTWARD from ring centre (was INWARD, hidden under cable hole).
- Bundle 3D STEP model from scottbez1/smartknob (Apache 2.0) so LEDs render
  in 3D. New libraries/oas.3dshapes/ with NOTICE.md for attribution.
- Add show_pin_labels option to gen_sk6812_side_pcb_footprint(); D11 gets
  vertical "Di"/"Gd" silk labels at pads 1/4 for visual orientation check
  during inspection.
- Per-LED radius overrides: D11/D15 R=11 (E-W axis symmetry), D12/D14
  R=16.5 (clear J1 mating plug), C21/C23 cap radial offset 2.6 mm (vs
  3.4 default) so caps sit OUTSIDE J1 plug no-go zone.

J1 (24V Phoenix terminal):
- Rotate Qwiic J9 180->0 (mating face faces south chord opening).
- Shift J1_PCB_Y +5 mm south to widen the plug clearance area.
- Add F.SilkS no-go rectangle (X=±8.73, Y=[+6.4,+21.5]) labelled "J1 PLUG"
  marking the area reserved for the mating plug. Component placement
  ensures nothing lies inside this rect.

F1 polyfuse:
- Downsize 2920 -> 1812 (Littelfuse 1812L075THDR, LCSC C262023) so the
  KiCad-stock R_1812_4532Metric.step can be used as the 3D body (CC-BY-SA
  + Design Exception, commitable to public repo). The stock 2920 footprint
  references a STEP file absent from KiCad 10 install.
- Add model_override parameter to _emit_stock_lib_footprint() helper to
  redirect (model ...) path when stock kicad_mod points at a missing file.

3D renders:
- Add 3 isometric views at 90/180/270 deg azimuth (in addition to existing
  iso = 0 deg) for full 360-deg visual review.

Layout follow-ups (all DRC clean):
- Move "J10 flash" silk text 3 mm south (D17 collision after radius bump).
- Increase MIKROE-2462 height/footprint half-extent entries to cover
  Fuse_1812_4532Metric footprint.
- Remove "AQI ring" board-level silk text (pads of D18 collided with
  the bbox after radius/rotation change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
Parts:
- F1: footprint Fuse:Fuse_2920_7451Metric -> Fuse:Fuse_1812_4532Metric; LCSC C207083 -> C262023; MPN 2920L075/60MR -> 1812L075THDR
Changed lines of the file:
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@@
 		)
 	)
-	(property "Footprint" "Fuse:Fuse_2920_7451Metric"
+	(property "Footprint" "Fuse:Fuse_1812_4532Metric"
 		(at 85.09 66.04 0)
 		(effects
@@
 			)
 		)
-		(property "MPN" "2920L075/60MR"
+		(property "MPN" "1812L075THDR"
 			(at 0 0 0)
 			(effects
@@
 			)
 		)
-		(property "LCSC" "C207083"
+		(property "LCSC" "C262023"
 			(at 0 0 0)
 			(effects

Commit message: fix(schematic): D1 TVS — D_Zener symbol replaces bidirectional D_TVS
SMBJ24A is a unidirectional TVS (verified via the A vs CA part-number
suffix convention and multiple distributor datasheets). D1 was drawn
with Device:D_TVS — KiCad's bidirectional TVS symbol (pins A1/A2, no
cathode). The netlist/iBOM described the part as "bidirectional" and
correct orientation relied solely on the angle=270 placement trick.

KiCad ships no unidirectional-TVS symbol; a unidirectional TVS shares
the Zener schematic glyph, so D1 now uses Device:D_Zener — self-
documenting K/A pins (pin 1 = K cathode binds canonically to D_SMB
pad 1 = cathode). Connectivity is unchanged; the net auto-name follows
the pin rename: Net-(D1-A1) -> Net-(D1-K).

Also delete the now-dead _sch_diode_tvs helper and the unused
Device:D_TVS lib_symbol block, and fix stale "angle=90" comments that
contradicted the actual angle=270 emit. oas_routes.py keeps the old
net name in its disabled autoroute chunks — already stale pending the
routing rework.

29/29 build PASS — DRC 0, ERC 0, determinism OK.

Co-Authored-By: Claude Opus 4.7 <noreply@anthropic.com>
Parts:
- D1: symbol Device:D_TVS -> Device:D_Zener
Changed lines of the file:
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@@
 )
 (symbol
-	(lib_id "Device:D_TVS")
+	(lib_id "Device:D_Zener")
 	(at 66.04 87.63 270)
 	(unit 1)
