File: hardware/kicad/mcu.kicad_sch (KiCad schematic)
At the start: 8 parts, among them J2 SWD/UART Recovery (DNP), J5 1x15 P2.54 mm female socket (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, J6 1x15 P2.54 mm female socket (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

Commit message: kicad: v0.25 - widen Mn3 back-fill regex to capture indented footprint blocks
Closes review-iteration-3 (Mn3-residual + Nt-doc-comment) at v0.24:

- _build_pcb_ref_to_footprint() regex (?m)^\(footprint "..." widened to
  (?m)^\s*\(footprint "..." . KiCad pretty-prints some (footprint ...) blocks
  in oas.kicad_pcb with leading tab/space indentation; the column-0 anchor
  silently skipped 31 of 76 placed footprints in v0.24, leaving 27 schematic
  real-component symbols with empty Footprint properties (ERC-silent but
  cosmetically wrong). Match count: 45 -> 76 (exactly equal to kiutils
  enumeration). Verified no nested (footprint "..." references exist.
- Inner re.match relaxed to re.search since sliced blocks can begin with
  whitespace.
- Docstring updated to disclose the regex behavior honestly (closes
  Nt-doc-comment from review iter-3).
- All 65 real-component schematic instances now carry a fully-qualified
  Lib:Name Footprint property. Empty-Footprint count: 0 (was 27 at v0.24,
  51 at v0.22). Previously-missed refs now lib-qualified: C2 + C5-C17, D1-D3,
  F1, L1-L2, R1-R7, plus ZT1-ZT4.
- DRC = 0/0, ERC = 0/0, determinism self-check passes (17 files bit-identical
  across two consecutive runs). PCB geometry unchanged - schematic-side
  .kicad_sch diffs only.
- Adds the iteration-3 review file (hardware/components/_review-iteration-3-v0.24.md).

Co-Authored-By: Claude Opus 4.7 (1M context) <noreply@anthropic.com>
Parts:
- C17: footprint (none) -> Capacitor_SMD:C_0603_1608Metric
- C9: footprint (none) -> Capacitor_SMD:C_0805_2012Metric
- R5, R6, R7: footprint (none) -> Resistor_SMD:R_0603_1608Metric
Changed lines of the file:
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@@
 		)
 	)
-	(property "Footprint" ""
+	(property "Footprint" "Capacitor_SMD:C_0805_2012Metric"
 		(at 129.54 80.01 0)
 		(effects
@@
 		)
 	)
-	(property "Footprint" ""
+	(property "Footprint" "Capacitor_SMD:C_0603_1608Metric"
 		(at 138.43 80.01 0)
 		(effects
@@
 		)
 	)
-	(property "Footprint" ""
+	(property "Footprint" "Resistor_SMD:R_0603_1608Metric"
 		(at 121.92 80.01 90)
 		(effects
@@
 		)
 	)
-	(property "Footprint" ""
+	(property "Footprint" "Resistor_SMD:R_0603_1608Metric"
 		(at 124.46 80.01 90)
 		(effects
@@
 		)
 	)
-	(property "Footprint" ""
+	(property "Footprint" "Resistor_SMD:R_0603_1608Metric"
 		(at 152.4 87.63 90)
 		(effects

Commit message: kicad+bom: v0.36 - swarm-audit fixes (4 CRITICAL + 3 IMPORTANT)
All 30-agent swarm audit findings from _swarm-audit-v0.35.md addressed.

CRITICAL fixes (would have caused board failure):
- C1 D1 TVS polarity: schematic angle 90→270 AND PCB rotation 0→180
  jointly land KiCad D_SMB pad 1 (cathode) on +24V VIN (was on GND).
  Net renamed Net-(D1-A2) → Net-(D1-A1) in oas_routes.py.
- C2 TPS62933 FB divider: schematic R2 44.2k→100k, R3 10k→30.9k for
  correct Vref=0.8V (was designed against wrong Vref=0.6V assumption).
  Vout = 0.8 × (1 + 100/30.9) = 3.39V (within ±3% of 3.3V target).
- C3 C7/C8 align: PCB-generator C7=22pF/C8=100nF (with swapped BST/SS
  roles) was contradicting the schematic C7=100nF BST + C8=47nF SS.
  Aligned PCB-generator to schematic (correct TPS62933 config).
- C4 Q1 substitution: PMV65XP (Vds=-20V) → AO3401A (LCSC C15127,
  Vds=-30V, same SOT-23 footprint). 8.9V margin over SMBJ24A 38.9V
  clamp. AO3401A drop-in: 1=G, 2=S, 3=D — no PCB layout change.

IMPORTANT fixes:
- I1 silk polarity markers: cathode bar on F.SilkS for D_SMA/D_SMB/
  D_SOD-323 (D1/D2/D3); "+" mark for CP_Radial (C1/C3/C4). Bar X
  computed from pad inner edge so silk clears mask opening by 0.25mm.
- I2 J10 cutout C3 north wall: +28.998 → +27.498 so pad 6 (BOOT)
  fully inside keepout (was 0.7mm outside).
- I3 J2/J10 DNP: (in_bom yes)→(in_bom no) when dnp flag is set.
- I7 D3 value text "500mW" → "200mW" matching BZT52C18S datasheet.

R1 value text aligned "100k" → "100k 1%" for consistent BOM grouping.

Verification: DRC=0, ERC=0, determinism PASS (17 files bit-identical),
Z-clearance PASS (76 footprints), preflight PASS, BOM=12 Basic + 11
Extended SMD + 8 THT (zero unmapped rows).

Co-Authored-By: Claude Opus 4.7 (1M context) <noreply@anthropic.com>
Parts:
- J2: now left out of the parts list
Changed lines of the file:
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@@
         		(unit 1)
         		(exclude_from_sim no)
-        		(in_bom yes)
+        		(in_bom no)
         		(on_board yes)
         		(dnp yes)

Commit message: kicad+bom: v0.38 - swarm audit v2 fixes (BOM-project coupling + silk polish)
30-agent read-only re-audit confirmed all v0.35-v0.37 CRITICAL fixes
in place and identified 6 follow-up items + 1 false positive. Applied
fixes:

Schematic ↔ BOM coupling (audit-16, primary user concern):
- generate.py: new _build_lcsc_metadata_map() + _apply_schematic_lcsc_metadata()
  injects Manufacturer / MPN / LCSC properties on every component symbol
  whose (Value, Footprint) matches a row in hardware/bom/lcsc-mapping.csv.
  Closes "projekt sobie, BOM sobie" — schematic is now self-sufficient
  for BOM export.
- export_production.py: BOM export switched to native kicad-cli --fields
  emitting Manufacturer + MPN columns directly from schematic. Post-process
  preserves them and adds JLCPCB_Library classification.
- New BOM CSV columns: Comment, Designator, Footprint, Manufacturer, MPN,
  LCSC, JLCPCB_Library, Qty.

Silkscreen polish (audit-26 / -27 / -24 / -28 / agent-08+11+30):
- D3 descriptor drift: 18V Zener → 10V Zener across generate.py PCB descr
  + 5 inline design comments (schematic Value + lcsc-mapping were already
  correct at v0.37; this fix syncs the source-of-truth comments).
- Radial cap "+" polarity marks: moved from pad_x+1.4 (INSIDE body radius,
  hidden post-assembly) to body_r+0.7 (~0.7 mm outside body, visible after
  the 8/6.3 mm cap solders down).
- SK6812 LED pin-1 dot: moved from F.Fab → F.SilkS in both lib generator
  and PCB-side footprint emitter, so the ring orientation is verifiable
  on physical PCB without consulting the assembly drawing.
- U1 LM2596S TO-263-5: added F.SilkS pin-1 dot at (-4.5, +1.5) radius 0.4
  for hand-assembly orientation.
- Board ID labels on F.SilkS: "Open Ambient Sensor" + "OAS v0.38" in the
  clear strip between MIKROE east edge (-12.7) and C3 cutout west (+4.9).
  Full repo URL on F.Fab (visible in renders, not silk-printed — URL too
  long for the strip at the 1.0 mm silk_min_text_height rule).

False positive confirmed (audit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
Parts:
- C17: LCSC (none) -> C14663; MPN (none) -> CC0603KRX7R9BB104; Manufacturer (none) -> Yageo
- C9: LCSC (none) -> C15850; MPN (none) -> CL21A106KAYNNNE; Manufacturer (none) -> Samsung Electro-Mechanics
- R5, R6: LCSC (none) -> C23162; MPN (none) -> 0603WAF4701T5E; Manufacturer (none) -> UNI-ROYAL (Uniroyal Elec)
- R7: LCSC (none) -> C25804; MPN (none) -> 0603WAF1002T5E; Manufacturer (none) -> UNI-ROYAL (Uniroyal Elec)
Changed lines of the file:
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@@
 		)
 	)
+		(property "Manufacturer" "Samsung Electro-Mechanics"
+			(at 0 0 0)
+			(effects
+				(font
+					(size 1.27 1.27)
+				)
+				(hide yes)
+			)
+		)
+		(property "MPN" "CL21A106KAYNNNE"
+			(at 0 0 0)
+			(effects
+				(font
+					(size 1.27 1.27)
+				)
+				(hide yes)
+			)
+		)
+		(property "LCSC" "C15850"
+			(at 0 0 0)
+			(effects
+				(font
+					(size 1.27 1.27)
+				)
+				(hide yes)
+			)
+		)
 	(pin "1"
 	)
@@
 		)
 	)
+		(property "Manufacturer" "Yageo"
+			(at 0 0 0)
+			(effects
+				(font
+					(size 1.27 1.27)
+				)
+				(hide yes)
+			)
+		)
+		(property "MPN" "CC0603KRX7R9BB104"
+			(at 0 0 0)
+			(effects
+				(font
+					(size 1.27 1.27)
+				)
+				(hide yes)
+			)
+		)
+		(property "LCSC" "C14663"
+			(at 0 0 0)
+			(effects
+				(font
+					(size 1.27 1.27)
+				)
+				(hide yes)
+			)
+		)
 	(pin "1"
 	)
@@
 		)
 	)
+		(property "Manufacturer" "UNI-ROYAL (Uniroyal Elec)"
+			(at 0 0 0)
+			(effects
+				(font
+					(size 1.27 1.27)
+				)
+				(hide yes)
+			)
+		)
+		(property "MPN" "0603WAF4701T5E"
+			(at 0 0 0)
+			(effects
+				(font
+					(size 1.27 1.27)
+				)
+				(hide yes)
+			)
+		)
+		(property "LCSC" "C23162"
+			(at 0 0 0)
+			(effects
+				(font
+					(size 1.27 1.27)
+				)
+				(hide yes)
+			)
+		)
 	(pin "1"
 	)
@@
 		)
 	)
+		(property "Manufacturer" "UNI-ROYAL (Uniroyal Elec)"
+			(at 0 0 0)
+			(effects
+				(font
+					(size 1.27 1.27)
+				)
+				(hide yes)
+			)
+		)
+		(property "MPN" "0603WAF4701T5E"
+			(at 0 0 0)
+			(effects
+				(font
+					(size 1.27 1.27)
+				)
+				(hide yes)
+			)
+		)
+		(property "LCSC" "C23162"
+			(at 0 0 0)
+			(effects
+				(font
+					(size 1.27 1.27)
+				)
+				(hide yes)
+			)
+		)
 	(pin "1"
 	)
@@
 		)
 	)
+		(property "Manufacturer" "UNI-ROYAL (Uniroyal Elec)"
+			(at 0 0 0)
+			(effects
+				(font
+					(size 1.27 1.27)
+				)
+				(hide yes)
+			)
+		)
+		(property "MPN" "0603WAF1002T5E"
+			(at 0 0 0)
+			(effects
+				(font
+					(size 1.27 1.27)
+				)
+				(hide yes)
+			)
+		)
+		(property "LCSC" "C25804"
+			(at 0 0 0)
+			(effects
+				(font
+					(size 1.27 1.27)
+				)
+				(hide yes)
+			)
+		)
 	(pin "1"
 	)
